File: mp3/mp3.kicad_pcb (KiCad board)
At the start: 2 copper layers, 32.1 x 53.2 mm, 33 parts, among them J1 USB4105-GF-A, J2 LEFT, J3 DEBUG, J4 RIGHT, U1 W25Q128JV, U2 RP2040, U3 MCP1702T-3302E_CB, Y1 12MHz

Commit message: fixed bypass cap gnd traces
Routing:
- net GND: track 40.2 -> 33.7 mm, vias 17 -> 22
